File: demos/pic_programmer/pic_programmer.kicad_pcb (KiCad board)
At the start: 2 copper layers, 160 x 99.1 mm, 63 parts, among them J1 DB9-FEMAL, P1 CONN_2, P101 CONN_1, P102 CONN_1, P103 CONN_1, P104 CONN_1, P105 CONN_1, P106 CONN_1, P2 SUPP28, P3 SUPP40, Q1 BC237, Q2 BC307, Q3 BC307, U1 24Cxx, U2 74HC125, U3 7805, U4 LT1373, U5 PIC_18_PINS, U6 PIC_8_PINS

Commit message: new changes
Parts:
- moved U3 35.8 mm to (91.7, 35.6)
Connections:
- net Net-(D11-A) renamed /neopolitan
- D11 pad 1: Net-(D11-K) -> /PC-DATA-IN-CAT
- J1 pad 8: /PC-DATA-IN -> /PC-DATA-IN-CAT
- Q1 pad 1: Net-(D11-K) -> /PC-DATA-IN-CAT
- R11 pad 1: Net-(D11-K) -> /PC-DATA-IN-CAT
- U2 pad 11: /PC-DATA-IN -> unconnected-(U2-Pad11)
Routing:
- net /PC-DATA-IN-CAT: track 0.00 -> 63.6 mm
- net /PC-DATA-IN: track 45.8 -> 0.00 mm
- net Net-(D11-K): track 17.8 -> 0.00 mm
Changed lines of the file:
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@@
 (kicad_pcb
-	(version 20260206)
+	(version 20260513)
 	(generator "pcbnew")
-	(generator_version "10.0")
+	(generator_version "10.99")
 	(general
 		(thickness 1.6)
@@
 	(layers
 		(0 "F.Cu" signal "top_layer")
-		(2 "B.Cu" signal "bottom_layer")
+		(2 "B.Cu" signal "mv")
 		(9 "F.Adhes" user "F.Adhesive")
 		(11 "B.Adhes" user "B.Adhesive")
@@
 				(epsilon_r 4.5)
 				(loss_tangent 0.02)
+				(spec_frequency 1000000000)
+				(dielectric_model constant)
 			)
 			(layer "B.Cu"
@@
 			(dashed_line_gap_ratio 3)
 			(svgprecision 6)
+			(pngdpi 300)
+			(pngantialias yes)
 			(plotframeref no)
 			(mode 1)
@@
 			(layers "*.Cu" "*.Mask")
 			(remove_unused_layers no)
-			(net "/PC-DATA-IN")
+			(net "unconnected-(U2-Pad11)")
 			(pintype "tri_state")
 		)
@@
 			(remove_unused_layers no)
 			(roundrect_rratio 0.15625)
-			(net "Net-(D11-K)")
+			(net "/PC-DATA-IN-CAT")
 			(pinfunction "K_1")
 			(pintype "passive")
@@
 			(layers "*.Cu" "*.Mask")
 			(remove_unused_layers no)
-			(net "Net-(D11-A)")
+			(net "/neopolitan")
 			(pinfunction "A_2")
 			(pintype "passive")
@@
 			(layers "*.Cu" "*.Mask")
 			(remove_unused_layers no)
-			(net "/PC-DATA-IN")
+			(net "/PC-DATA-IN-CAT")
 			(pinfunction "P8_8")
 			(pintype "passive")
@@
 			(remove_unused_layers no)
 			(roundrect_rratio 0.25)
-			(net "Net-(D11-K)")
+			(net "/PC-DATA-IN-CAT")
 			(pinfunction "C_1")
 			(pintype "passive")
@@
 			(layers "*.Cu" "*.Mask")
 			(remove_unused_layers no)
-			(net "Net-(D11-A)")
+			(net "/neopolitan")
 			(pintype "passive")
 		)
@@
 	(footprint "Package_TO_SOT_THT:TO-220-3_Horizontal_TabDown"
 		(layer "F.Cu")
-		(at 96.52 71.12)
+		(at 91.66 35.63)
 		(descr "TO-220-3, Horizontal, RM 2.54mm, see https://www.vishay.com/docs/66542/to-220-1.pdf, generated with kicad-footprint-generator TO_SOT_THT_generate.py")
 		(tags "TO-220-3 Horizontal RM 2.54mm")
@@
 			(layers "*.Cu" "*.Mask")
 			(remove_unused_layers no)
-			(net "Net-(D11-K)")
+			(net "/PC-DATA-IN-CAT")
 			(pintype "passive")
 		)
@@
 		(width 0.5)
 		(layer "B.Cu")
-		(net "/PC-DATA-IN")
+		(net "/PC-DATA-IN-CAT")
 	)
 	(segment
@@
 		(width 0.5)
 		(layer "B.Cu")
-		(net "/PC-DATA-IN")
+		(net "/PC-DATA-IN-CAT")
 	)
 	(segment
@@
 		(width 0.5)
 		(layer "B.Cu")
-		(net "/PC-DATA-IN")
+		(net "/PC-DATA-IN-CAT")
+	)
+	(segment
+		(start 141.605 72.517)
+		(end 140.081 70.993)
+		(width 0.5)
+		(layer "B.Cu")
+		(net "/PC-DATA-IN-CAT")
 	)
 	(segment
@@
 		(width 0.5)
 		(layer "B.Cu")
-		(net "/PC-DATA-IN")
+		(net "/PC-DATA-IN-CAT")
 	)
 	(segment
@@
 		(width 0.5)
 		(layer "B.Cu")
-		(net "/PC-DATA-IN")
+		(net "/PC-DATA-IN-CAT")
 	)
 	(segment
@@
 		(width 0.5)
 		(layer "B.Cu")
-		(net "/PC-DATA-IN")
+		(net "/PC-DATA-IN-CAT")
 	)
 	(segment
@@
 		(width 0.5)
 		(layer "B.Cu")
-		(net "/PC-DATA-IN")
+		(net "/PC-DATA-IN-CAT")
 	)
 	(segment
@@
 		(width 0.5)
 		(layer "B.Cu")
-		(net "/PC-DATA-IN")
+		(net "/PC-DATA-IN-CAT")
 	)
 	(segment
@@
 		(width 0.5)
 		(layer "B.Cu")
-		(net "/PC-DATA-IN")
-	)
-	(segment
-		(start 109.174001 113.217001)
-		(end 109.234002 113.157)
-		(width 0.5)
-		(layer "B.Cu")
-		(net "/PC-DATA-IN")
+		(net "/PC-DATA-IN-CAT")
 	)
 	(segment
-		(start 109.234002 113.157)
-		(end 111.887 113.157)
+		(start 141.605 78.105)
+		(end 141.605 72.517)
 		(width 0.5)
 		(layer "B.Cu")
-		(net "/PC-DATA-IN")
+		(net "/PC-DATA-IN-CAT")
 	)
 	(segment
-		(start 100.954001 113.187001)
-		(end 100.984002 113.157)
+		(start 141.224 69.85)
+		(end 146.05 69.85)
 		(width 0.5)
 		(layer "B.Cu")
-		(net "/PC-DATA-IN")
+		(net "/PC-DATA-IN-CAT")
 	)
 	(segment
-		(start 99.705999 113.187001)
-		(end 100.954001 113.187001)
+		(start 109.174001 113.217001)
+		(end 109.234002 113.157)
 		(width 0.5)
 		(layer "B.Cu")
-		(net "/PC-DATA-IN")
+		(net "/PC-DATA-IN-CAT")
 	)
 	(segment
-		(start 99.675998 113.157)
-		(end 99.705999 113.187001)
+		(start 109.234002 113.157)
+		(end 111.887 113.157)
 		(width 0.5)
 		(layer "B.Cu")
-		(net "/PC-DATA-IN")
+		(net "/PC-DATA-IN-CAT")
 	)
 	(segment
-		(start 111.887 113.157)
-		(end 113.03 114.3)
+		(start 140.081 70.993)
+		(end 141.224 69.85)
 		(width 0.5)
 		(layer "B.Cu")
-		(net "/PC-DATA-IN")
+		(net "/PC-DATA-IN-CAT")
 	)
 	(segment
-		(start 83.425 113.275)
-		(end 79.76 113.275)
+		(start 100.954001 113.187001)
+		(end 100.984002 113.157)
 		(width 0.5)
 		(layer "B.Cu")
-		(net "/PC-DATA-IN")
+		(net "/PC-DATA-IN-CAT")
 	)
 	(segment
-		(start 141.605 72.517)
-		(end 140.081 70.993)
+		(start 99.705999 113.187001)
+		(end 100.954001 113.187001)
 		(width 0.5)
 		(layer "B.Cu")
-		(net "Net-(D11-K)")
+		(net "/PC-DATA-IN-CAT")
 	)
 	(segment
-		(start 141.605 78.105)
-		(end 141.605 72.517)
+		(start 99.675998 113.157)
+		(end 99.705999 113.187001)
 		(width 0.5)
 		(layer "B.Cu")
-		(net "Net-(D11-K)")
+		(net "/PC-DATA-IN-CAT")
 	)
 	(segment
-		(start 141.224 69.85)
-		(end 146.05 69.85)
+		(start 111.887 113.157)
+		(end 113.03 114.3)
 		(width 0.5)
 		(layer "B.Cu")
-		(net "Net-(D11-K)")
+		(net "/PC-DATA-IN-CAT")
 	)
 	(segment
-		(start 140.081 70.993)
-		(end 141.224 69.85)
+		(start 139.065 80.645)
+		(end 141.605 78.105)
 		(width 0.5)
 		(layer "B.Cu")
-		(net "Net-(D11-K)")
+		(net "/PC-DATA-IN-CAT")
 	)
 	(segment
-		(start 139.065 80.645)
-		(end 141.605 78.105)
+		(start 83.425 113.275)
+		(end 79.76 113.275)
 		(width 0.5)
 		(layer "B.Cu")
-		(net "Net-(D11-K)")
+		(net "/PC-DATA-IN-CAT")
 	)
 	(segment
@@
 		(width 0.5)
 		(layer "B.Cu")
-		(net "Net-(D11-A)")
+		(net "/neopolitan")
 	)
 	(segment
@@
 		(width 0.5)
 		(layer "B.Cu")
-		(net "Net-(D11-A)")
+		(net "/neopolitan")
 	)
 	(segment
@@
 		(width 0.5)
 		(layer "B.Cu")
-		(net "Net-(D11-A)")
+		(net "/neopolitan")
 	)
 	(segment
