File: demos/pic_programmer/pic_programmer.kicad_pcb (KiCad board)
At the start: 2 copper layers, 160 x 99.1 mm, 63 parts, among them J1 DB9-FEMAL, P1 CONN_2, P101 CONN_1, P102 CONN_1, P103 CONN_1, P104 CONN_1, P105 CONN_1, P106 CONN_1, P2 SUPP28, P3 SUPP40, Q1 BC237, Q2 BC307, Q3 BC307, U1 24Cxx, U2 74HC125, U3 7805, U4 LT1373, U5 PIC_18_PINS, U6 PIC_8_PINS

Commit message: Works-Like Prototype
Conduit Schematic + Site Layout conduit system, works-like prototype:
- Routing: spec-gated, local-board-frame 22.5 snapping, filleted bends (faulty if radius doesn't fit), live clearance/bend warnings, layer picker (auto from net-class name), termination highlight
- Node editing: double-click on conduit; angle-preserving edits (move nearest node, error-state if invalid); right-click delete node/section/anchor/route; table editor reachable from right-click
- Equipment anchors: bind endpoint to footprint, follow on move (EditRouteNode rule), endpoint change drops anchor, faulty/dashed state
- Conduit Depths: layers tied to real copper layers, add (pairs) / delete-selected, per-layer depth + display name
- Cable Specs: per-class + per-net + editable Cable Types panel; net-class resolution via effective (assigned) class
- Conduit color = layer color; no-spec box outlined red; total-bend shown in box (red >360)
- Exports: Circuit List + Raceway List CSV (length, total bend, per-type bend counts, fill%)
- Conduit pickers sorted natural-numeric

Co-Authored-By: Claude Opus 4.8 <noreply@anthropic.com>
Parts:
- moved U3 38.3 mm to (129.3, 28.5)
Changed lines of the file:
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@@
 	(footprint "Package_TO_SOT_THT:TO-220-3_Horizontal_TabDown"
 		(layer "F.Cu")
-		(at 91.66 35.63)
+		(at 129.26 28.46)
 		(descr "TO-220-3, Horizontal, RM 2.54mm, see https://www.vishay.com/docs/66542/to-220-1.pdf, generated with kicad-footprint-generator TO_SOT_THT_generate.py")
 		(tags "TO-220-3 Horizontal RM 2.54mm")
