File: demos/pic_programmer/pic_programmer.kicad_sch (KiCad schematic)
At the start: 56 parts, among them J1 DB9-FEMAL, P1 CONN_2, P101 CONN_1, P102 CONN_1, P103 CONN_1, P104 CONN_1, P105 CONN_1, P106 CONN_1, Q1 BC237, Q2 BC307, Q3 BC307, U2 74HC125, U3 7805, U4 LT1373

Commit message: new changes
Connections:
- net PC-DATA-IN-CAT: now reaches D11.1 (K), Q1.1 (C), R11.1
- net PC-DATA-IN-CAT: now also J1.8 (P8)
- net neopolitan: now reaches D11.2 (A), R19.1
- net PC-DATA-IN: no longer names the net of U2.11
- net PC-DATA-IN: no longer J1.8 (P8)
Changed lines of the file:
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@@
 (kicad_sch
-	(version 20260101)
+	(version 20260512)
 	(generator "eeschema")
-	(generator_version "10.0")
+	(generator_version "10.99")
 	(paper "A4")
 	(title_block
@@
 	)
 	(junction
+		(at 186.69 73.66)
+		(diameter 0)
+		(color 0 0 0 0)
+	)
+	(junction
 		(at 154.94 31.75)
 		(diameter 1.016)
@@
 		(diameter 1.016)
 		(color 0 0 0 0)
+	)
+	(junction
+		(at 168.91 73.66)
+		(diameter 0)
+		(color 0 0 0 0)
+	)
+	(no_connect
+		(at 43.18 81.28)
+	)
+	(no_connect
+		(at 43.18 83.82)
 	)
 	(no_connect
@@
 	)
 	(no_connect
-		(at 43.18 81.28)
-	)
-	(no_connect
 		(at 43.18 86.36)
 	)
@@
 	)
 	(no_connect
-		(at 43.18 83.82)
-	)
-	(no_connect
 		(at 171.45 143.51)
 	)
@@
 	(wire
 		(pts
-			(xy 102.87 106.68) (xy 57.15 106.68)
-		)
-		(stroke
-			(width 0)
-			(type solid)
-		)
-	)
-	(wire
-		(pts
 			(xy 250.19 156.21) (xy 243.84 156.21)
 		)
@@
 	(wire
 		(pts
-			(xy 57.15 106.68) (xy 57.15 93.98)
-		)
-		(stroke
-			(width 0)
-			(type solid)
-		)
-	)
-	(wire
-		(pts
 			(xy 250.19 143.51) (xy 243.84 143.51)
 		)
@@
 	(wire
 		(pts
+			(xy 168.91 73.66) (xy 177.8 73.66)
+		)
+		(stroke
+			(width 0)
+			(type solid)
+		)
+	)
+	(wire
+		(pts
 			(xy 144.78 19.05) (xy 154.94 19.05)
 		)
@@
 	(wire
 		(pts
-			(xy 148.59 73.66) (xy 177.8 73.66)
+			(xy 148.59 73.66) (xy 168.91 73.66)
 		)
 		(stroke
@@
 	(wire
 		(pts
+			(xy 102.87 104.14) (xy 57.15 104.14)
+		)
+		(stroke
+			(width 0)
+			(type solid)
+		)
+	)
+	(wire
+		(pts
 			(xy 187.96 67.31) (xy 190.5 67.31)
 		)
@@
 	(wire
 		(pts
+			(xy 57.15 104.14) (xy 57.15 93.98)
+		)
+		(stroke
+			(width 0)
+			(type solid)
+		)
+	)
+	(wire
+		(pts
+			(xy 186.69 71.12) (xy 186.69 73.66)
+		)
+		(stroke
+			(width 0)
+			(type solid)
+		)
+	)
+	(wire
+		(pts
 			(xy 233.68 160.02) (xy 233.68 152.4)
 		)
@@
 	(wire
 		(pts
+			(xy 168.91 95.25) (xy 168.91 73.66)
+		)
+		(stroke
+			(width 0)
+			(type solid)
+		)
+	)
+	(wire
+		(pts
 			(xy 144.78 19.05) (xy 144.78 21.59)
 		)
@@
 	(wire
 		(pts
+			(xy 186.69 73.66) (xy 190.5 73.66)
+		)
+		(stroke
+			(width 0)
+			(type solid)
+		)
+	)
+	(wire
+		(pts
 			(xy 194.31 81.28) (xy 196.85 81.28)
 		)
@@
 	(wire
 		(pts
-			(xy 190.5 73.66) (xy 185.42 73.66)
-		)
-		(stroke
-			(width 0)
-			(type solid)
-		)
-	)
-	(wire
-		(pts
 			(xy 81.28 168.91) (xy 81.28 171.45)
 		)
@@
 	(wire
 		(pts
+			(xy 102.87 95.25) (xy 168.91 95.25)
+		)
+		(stroke
+			(width 0)
+			(type solid)
+		)
+	)
+	(wire
+		(pts
 			(xy 97.79 129.54) (xy 97.79 133.35)
 		)
@@
 	(wire
 		(pts
+			(xy 186.69 73.66) (xy 185.42 73.66)
+		)
+		(stroke
+			(width 0)
+			(type solid)
+		)
+	)
+	(wire
+		(pts
 			(xy 223.52 130.81) (xy 222.25 130.81)
 		)
@@
 	(wire
 		(pts
+			(xy 102.87 104.14) (xy 102.87 95.25)
+		)
+		(stroke
+			(width 0)
+			(type solid)
+		)
+	)
+	(wire
+		(pts
 			(xy 238.76 143.51) (xy 222.25 143.51)
 		)
@@
 			(width 0)
 			(type dash)
+		)
+	)
+	(label "neopolitan"
+		(at 186.69 71.12 0)
+		(effects
+			(font
+				(size 1.27 1.27)
+			)
+			(justify left bottom)
 		)
 	)
@@
 		)
 	)
-	(label "PC-DATA-IN"
-		(at 68.58 106.68 0)
+	(label "PC-DATA-IN-CAT"
+		(at 69.85 104.14 0)
 		(effects
 			(font
